File: Hardware/NomiMatrix_2/NomiMatrix_2.kicad_sch (KiCad schematic)
At the start: 0 parts

Commit message: recreated basic matrix
Parts:
- added D1, D10, D100, D11, D12, D13, D14, D15, D16, D17, D18, D19, D2, D20, D21, D22, D23, D24, D25, D26, D27, D28, D29, D3, D30, D31, D32, D33, D34, D35, D36, D37, D38, D39, D4, D40, D41, D42, D43, D44, D45, D46, D47, D48, D49, D5, D50, D51, D52, D53, D54, D55, D56, D57, D58, D59, D6, D60, D61, D62, D63, D64, D65, D66, D67, D68, D69, D7, D70, D71, D72, D73, D74, D75, D76, D77, D78, D79, D8, D80, D81, D82, D83, D84, D85, D86, D87, D88, D89, D9, D90, D91, D92, D93, D94, D95, D96, D97, D98, D99: WS2812B, LED_SMD:LED_WS2812B_PLCC4_5.0x5.0mm_P3.2mm, symbol LED:WS2812B
Connections:
- new net: D63.2 (DOUT), D67.4 (DIN)
- new net: D59.2 (DOUT), D63.4 (DIN)
- new net: D95.2 (DOUT), D97.4 (DIN)
- new net: D93.2 (DOUT), D95.4 (DIN)
- new net: D13.2 (DOUT), D14.4 (DIN)
- new net: D12.2 (DOUT), D13.4 (DIN)
- new net: D41.2 (DOUT), D45.4 (DIN)
- new net: D40.2 (DOUT), D41.4 (DIN)
- new net: D86.2 (DOUT), D88.4 (DIN)
- new net: D84.2 (DOUT), D86.4 (DIN)
- new net: D32.2 (DOUT), D34.4 (DIN)
- new net: D30.2 (DOUT), D32.4 (DIN)
- new net: D29.2 (DOUT), D31.4 (DIN)
- new net: D27.2 (DOUT), D29.4 (DIN)
- new net: D97.2 (DOUT), D99.4 (DIN)
- new net: D64.2 (DOUT), D68.4 (DIN)
- new net: D60.2 (DOUT), D64.4 (DIN)
- new net: D57.2 (DOUT), D61.4 (DIN)
- new net: D53.2 (DOUT), D57.4 (DIN)
- new net: D28.2 (DOUT), D30.4 (DIN)
- new net: D50.2 (DOUT), D54.4 (DIN)
- new net: D46.2 (DOUT), D50.4 (DIN)
- new net: D3.2 (DOUT), D4.4 (DIN)
- new net: D2.2 (DOUT), D3.4 (DIN)
- new net: D45.2 (DOUT), D49.4 (DIN)
- new net: D61.2 (DOUT), D65.4 (DIN)
- new net: D49.2 (DOUT), D53.4 (DIN)
- new net: D23.2 (DOUT), D25.4 (DIN)
- new net: D21.2 (DOUT), D23.4 (DIN)
- new net: D44.2 (DOUT), D48.4 (DIN)
- new net: D44.4 (DIN), D79.2 (DOUT)
- new net: D22.2 (DOUT), D24.4 (DIN)
- new net: D22.4 (DIN), D39.2 (DOUT)
- new net: D94.2 (DOUT), D96.4 (DIN)
- new net: D92.2 (DOUT), D94.4 (DIN)
- new net: D31.2 (DOUT), D33.4 (DIN)
- new net: D17.2 (DOUT), D18.4 (DIN)
- new net: D16.2 (DOUT), D17.4 (DIN)
- new net: D58.2 (DOUT), D62.4 (DIN)
- new net: D54.2 (DOUT), D58.4 (DIN)
- new net: D19.2 (DOUT), D20.4 (DIN)
- new net: D18.2 (DOUT), D19.4 (DIN)
- new net: D36.2 (DOUT), D38.4 (DIN)
- new net: D34.2 (DOUT), D36.4 (DIN)
- new net: D82.4 (DIN), D99.2 (DOUT)
- new net: D89.2 (DOUT), D91.4 (DIN)
- new net: D87.2 (DOUT), D89.4 (DIN)
- new net: D10.2 (DOUT), D11.4 (DIN)
- new net: D10.4 (DIN), D9.2 (DOUT)
- new net: D4.2 (DOUT), D5.4 (DIN)
- new net: D6.2 (DOUT), D7.4 (DIN)
- new net: D5.2 (DOUT), D6.4 (DIN)
- new net: D37.2 (DOUT), D39.4 (DIN)
- new net: D35.2 (DOUT), D37.4 (DIN)
- new net: D100.4 (DIN), D98.2 (DOUT)
- new net: D96.2 (DOUT), D98.4 (DIN)
- new net: D33.2 (DOUT), D35.4 (DIN)
- new net: D20.2 (DOUT), D21.4 (DIN)
- new net: D1.2 (DOUT), D2.4 (DIN)
- new net: D43.4 (DIN), D78.2 (DOUT)
- new net: D74.2 (DOUT), D78.4 (DIN)
- new net: D81.2 (DOUT), D83.4 (DIN)
- new net: D80.2 (DOUT), D81.4 (DIN)
- new net: D14.2 (DOUT), D15.4 (DIN)
- new net: D52.2 (DOUT), D56.4 (DIN)
- new net: D48.2 (DOUT), D52.4 (DIN)
- new net: D72.2 (DOUT), D76.4 (DIN)
- new net: D68.2 (DOUT), D72.4 (DIN)
- new net: D25.2 (DOUT), D27.4 (DIN)
- new net: D85.2 (DOUT), D87.4 (DIN)
- new net: D66.2 (DOUT), D70.4 (DIN)
- new net: D62.2 (DOUT), D66.4 (DIN)
- new net: D71.2 (DOUT), D75.4 (DIN)
- new net: D67.2 (DOUT), D71.4 (DIN)
- new net: D42.2 (DOUT), D46.4 (DIN)
- new net: D42.4 (DIN), D77.2 (DOUT)
- new net: D90.2 (DOUT), D92.4 (DIN)
- new net: D82.2 (DOUT), D84.4 (DIN)
- new net: D15.2 (DOUT), D16.4 (DIN)
- new net: D7.2 (DOUT), D8.4 (DIN)
- new net: D11.2 (DOUT), D12.4 (DIN)
- new net: D38.2 (DOUT), D40.4 (DIN)
- new net: D76.2 (DOUT), D80.4 (DIN)
- new net: D70.2 (DOUT), D74.4 (DIN)
- new net: D83.2 (DOUT), D85.4 (DIN)
- new net: D91.2 (DOUT), D93.4 (DIN)
- new net: D73.2 (DOUT), D77.4 (DIN)
- new net: D24.2 (DOUT), D26.4 (DIN)
- new net: D55.2 (DOUT), D59.4 (DIN)
- new net: D51.2 (DOUT), D55.4 (DIN)
- new net: D56.2 (DOUT), D60.4 (DIN)
- new net: D47.2 (DOUT), D51.4 (DIN)
- new net: D43.2 (DOUT), D47.4 (DIN)
- new net: D26.2 (DOUT), D28.4 (DIN)
- new net: D69.2 (DOUT), D73.4 (DIN)
- new net: D88.2 (DOUT), D90.4 (DIN)
- new net: D75.2 (DOUT), D79.4 (DIN)
- new net: D8.2 (DOUT), D9.4 (DIN)
- new net: D65.2 (DOUT), D69.4 (DIN)
- new net +5V: D1.1 (VDD), D10.1 (VDD), D100.1 (VDD), D11.1 (VDD), D12.1 (VDD), D13.1 (VDD), D14.1 (VDD), D15.1 (VDD), D16.1 (VDD), D17.1 (VDD), D18.1 (VDD), D19.1 (VDD), D2.1 (VDD), D20.1 (VDD), D21.1 (VDD), D22.1 (VDD), D23.1 (VDD), D24.1 (VDD), D25.1 (VDD), D26.1 (VDD), D27.1 (VDD), D28.1 (VDD), D29.1 (VDD), D3.1 (VDD), D30.1 (VDD), D31.1 (VDD), D32.1 (VDD), D33.1 (VDD), D34.1 (VDD), D35.1 (VDD), D36.1 (VDD), D37.1 (VDD), D38.1 (VDD), D39.1 (VDD), D4.1 (VDD), D40.1 (VDD), D41.1 (VDD), D42.1 (VDD), D43.1 (VDD), D44.1 (VDD), D45.1 (VDD), D46.1 (VDD), D47.1 (VDD), D48.1 (VDD), D49.1 (VDD), D5.1 (VDD), D50.1 (VDD), D51.1 (VDD), D52.1 (VDD), D53.1 (VDD), D54.1 (VDD), D55.1 (VDD), D56.1 (VDD), D57.1 (VDD), D58.1 (VDD), D59.1 (VDD), D6.1 (VDD), D60.1 (VDD), D61.1 (VDD), D62.1 (VDD), D63.1 (VDD), D64.1 (VDD), D65.1 (VDD), D66.1 (VDD), D67.1 (VDD), D68.1 (VDD), D69.1 (VDD), D7.1 (VDD), D70.1 (VDD), D71.1 (VDD), D72.1 (VDD), D73.1 (VDD), D74.1 (VDD), D75.1 (VDD), D76.1 (VDD), D77.1 (VDD), D78.1 (VDD), D79.1 (VDD), D8.1 (VDD), D80.1 (VDD), D81.1 (VDD), D82.1 (VDD), D83.1 (VDD), D84.1 (VDD), D85.1 (VDD), D86.1 (VDD), D87.1 (VDD), D88.1 (VDD), D89.1 (VDD), D9.1 (VDD), D90.1 (VDD), D91.1 (VDD), D92.1 (VDD), D93.1 (VDD), D94.1 (VDD), D95.1 (VDD), D96.1 (VDD), D97.1 (VDD), D98.1 (VDD), D99.1 (VDD)
- new net GND: D1.3 (VSS), D10.3 (VSS), D100.3 (VSS), D11.3 (VSS), D12.3 (VSS), D13.3 (VSS), D14.3 (VSS), D15.3 (VSS), D16.3 (VSS), D17.3 (VSS), D18.3 (VSS), D19.3 (VSS), D2.3 (VSS), D20.3 (VSS), D21.3 (VSS), D22.3 (VSS), D23.3 (VSS), D24.3 (VSS), D25.3 (VSS), D26.3 (VSS), D27.3 (VSS), D28.3 (VSS), D29.3 (VSS), D3.3 (VSS), D30.3 (VSS), D31.3 (VSS), D32.3 (VSS), D33.3 (VSS), D34.3 (VSS), D35.3 (VSS), D36.3 (VSS), D37.3 (VSS), D38.3 (VSS), D39.3 (VSS), D4.3 (VSS), D40.3 (VSS), D41.3 (VSS), D42.3 (VSS), D43.3 (VSS), D44.3 (VSS), D45.3 (VSS), D46.3 (VSS), D47.3 (VSS), D48.3 (VSS), D49.3 (VSS), D5.3 (VSS), D50.3 (VSS), D51.3 (VSS), D52.3 (VSS), D53.3 (VSS), D54.3 (VSS), D55.3 (VSS), D56.3 (VSS), D57.3 (VSS), D58.3 (VSS), D59.3 (VSS), D6.3 (VSS), D60.3 (VSS), D61.3 (VSS), D62.3 (VSS), D63.3 (VSS), D64.3 (VSS), D65.3 (VSS), D66.3 (VSS), D67.3 (VSS), D68.3 (VSS), D69.3 (VSS), D7.3 (VSS), D70.3 (VSS), D71.3 (VSS), D72.3 (VSS), D73.3 (VSS), D74.3 (VSS), D75.3 (VSS), D76.3 (VSS), D77.3 (VSS), D78.3 (VSS), D79.3 (VSS), D8.3 (VSS), D80.3 (VSS), D81.3 (VSS), D82.3 (VSS), D83.3 (VSS), D84.3 (VSS), D85.3 (VSS), D86.3 (VSS), D87.3 (VSS), D88.3 (VSS), D89.3 (VSS), D9.3 (VSS), D90.3 (VSS), D91.3 (VSS), D92.3 (VSS), D93.3 (VSS), D94.3 (VSS), D95.3 (VSS), D96.3 (VSS), D97.3 (VSS), D98.3 (VSS), D99.3 (VSS)

Commit message: Added an USB and the microcontroller chip, that will be used (becuase I have a lot of them)
Parts:
- added J1, J2: Conn_01x03, symbol Connector_Generic:Conn_01x03
- added J3: USB_C_Receptacle_USB2.0_16P, symbol Connector:USB_C_Receptacle_USB2.0_16P
- added R1: 33K, symbol Device:R
- added R2: 82K, symbol Device:R
- added U1: STM32F373CBTx, Package_QFP:LQFP-48_7x7mm_P0.5mm, symbol MCU_ST_STM32F3:STM32F373CBTx
Connections:
- net +5V: now also J1.1 (Pin_1), J2.1 (Pin_1), J3.A4 (VBUS), J3.A9 (VBUS), J3.B4 (VBUS), J3.B9 (VBUS), R1.1
- net GND: now also J1.3 (Pin_3), J2.3 (Pin_3), J3.A1 (GND), J3.A12 (GND), J3.B1 (GND), J3.B12 (GND), J3.S1 (SHIELD), R2.2, U1.47 (VSS)
- net at D1.4 (DIN): now also J1.2 (Pin_2)
- net at D100.2 (DOUT): now also J2.2 (Pin_2)
- new net +3.3V: R1.2, R2.1, U1.17 (VDD), U1.48 (VDD)
